File: KiCAD/KZ80-USBKBD.sch (KiCad schematic (older format))
At the start: 33 parts, among them J1 SBC8080 BUS, J2 CON-A, J3 CMT-OUT, J4 232C(DEBUG), J5 ADR-JP2, J6 ADR-JP1, SW1 SW_SPST, U1 Pico, U2 8255, U3 74HC139, U4 74HC00

Commit message: LEDフットプリント間違い修正
Parts:
- D1, D2: footprint LED_THT:LED_D3.0mm-3 -> LED_THT:LED_D3.0mm
Changed lines of the file:
@@
 F 0 "D1" H 3743 4866 50  0000 C CNN
 F 1 "KANA LED" H 3743 4775 50  0000 C CNN
-F 2 "LED_THT:LED_D3.0mm-3" H 3750 4650 50  0001 C CNN
+F 2 "LED_THT:LED_D3.0mm" H 3750 4650 50  0001 C CNN
 F 3 "~" H 3750 4650 50  0001 C CNN
 	1    3750 4650
@@
 F 0 "D2" H 3743 5266 50  0000 C CNN
 F 1 "CAPS LED" H 3743 5175 50  0000 C CNN
-F 2 "LED_THT:LED_D3.0mm-3" H 3750 5050 50  0001 C CNN
+F 2 "LED_THT:LED_D3.0mm" H 3750 5050 50  0001 C CNN
 F 3 "~" H 3750 5050 50  0001 C CNN
 	1    3750 5050
